Commit message: Add bulk of functionality

File: src/ros1_examples/descriptions/_d435.urdf.xacro (robot description, xacro)
@@ -45,5 +45,5 @@
       <origin xyz="${d435_cam_mount_from_center_offset} ${-d435_cam_depth_py} 0" rpy="${M_PI/2} 0 ${M_PI/2}"/>
         <geometry>
-	        <mesh filename="package://ros_demos/meshes/d435.dae" />
+	        <mesh filename="package://ros1_examples/meshes/d435.dae" />
         </geometry>
         <material name="${name}_aluminum"/>

File: src/ros1_examples/descriptions/slamcore-kobuki.urdf.xacro (robot description, xacro)
@@ -9,5 +9,5 @@
   <xacro:arg name="camera_link_frame_rpy" default=""/>
   <xacro:include filename="$(find kobuki_description)/urdf/kobuki.urdf.xacro" />
-  <xacro:include filename="$(find ros_demos)/descriptions/_d435.urdf.xacro" />
+  <xacro:include filename="$(find ros1_examples)/descriptions/_d435.urdf.xacro" />
   <xacro:kobuki/>
   <xacro:sensor_d435 name="$(arg camera_tf_root)" parent="base_link">

Commit message: [MISC] Trim realsense xacro file
Since we're publishing most of the realsense frames ourselves, we don't
need to publish these frames as part of the realsense URDF file. This
removes the extra to simplify the overall TF tree.

File: src/ros1_examples/descriptions/_d435.urdf.xacro (robot description, xacro)
@@ -62,56 +62,4 @@
       </inertial>
     </link>
-    <!-- camera depth joints and links -->
-    <joint name="${name}_depth_joint" type="fixed">
-      <origin xyz="0 0 0" rpy="0 0 0"/>
-      <parent link="${name}_link"/>
-      <child link="${name}_depth_frame" />
-    </joint>
-    <link name="${name}_depth_frame"/>
-    <joint name="${name}_depth_optical_joint" type="fixed">
-      <origin xyz="0 0 0" rpy="${-M_PI/2} 0 ${-M_PI/2}" />
-      <parent link="${name}_depth_frame" />
-      <child link="${name}_depth_optical_frame" />
-    </joint>
-    <link name="${name}_depth_optical_frame"/>
-    <!-- camera left IR joints and links -->
-    <joint name="${name}_left_ir_joint" type="fixed">
-      <origin xyz="0 ${d435_cam_depth_to_left_ir_offset} 0" rpy="0 0 0" />
-      <parent link="${name}_depth_frame" />
-      <child link="${name}_left_ir_frame" />
-    </joint>
-    <link name="${name}_left_ir_frame"/>
-    <joint name="${name}_left_ir_optical_joint" type="fixed">
-      <origin xyz="0 0 0" rpy="${-M_PI/2} 0 ${-M_PI/2}" />
-      <parent link="${name}_left_ir_frame" />
-      <child link="${name}_left_ir_optical_frame" />
-    </joint>
-    <link name="${name}_left_ir_optical_frame"/>
-    <!-- camera right IR joints and links -->
-    <joint name="${name}_right_ir_joint" type="fixed">
-      <origin xyz="0 ${d435_cam_depth_to_right_ir_offset} 0" rpy="0 0 0" />
-      <parent link="${name}_depth_frame" />
-      <child link="${name}_right_ir_frame" />
-    </joint>
-    <link name="${name}_right_ir_frame"/>
-    <joint name="${name}_right_ir_optical_joint" type="fixed">
-      <origin xyz="0 0 0" rpy="${-M_PI/2} 0 ${-M_PI/2}" />
-      <parent link="${name}_right_ir_frame" />
-      <child link="${name}_right_ir_optical_frame" />
-    </joint>
-    <link name="${name}_right_ir_optical_frame"/>
-    <!-- camera color joints and links -->
-    <joint name="${name}_color_joint" type="fixed">
-      <origin xyz="0 ${d435_cam_depth_to_color_offset} 0" rpy="0 0 0" />
-      <parent link="${name}_depth_frame" />
-      <child link="${name}_color_frame" />
-    </joint>
-    <link name="${name}_color_frame"/>
-    <joint name="${name}_color_optical_joint" type="fixed">
-      <origin xyz="0 0 0" rpy="${-M_PI/2} 0 ${-M_PI/2}" />
-      <parent link="${name}_color_frame" />
-      <child link="${name}_color_optical_frame" />
-    </joint>
-    <link name="${name}_color_optical_frame"/>
   </xacro:macro>
 </robot>
