Commit message: [SCS-2659] Make CAMERA_LINK_FRAME_* variables refer to the SLAMcore transform.
Until now the CAMERA_LINK_FRAME_* would determine the position of the
realsense URDF file and not the pose of the SLAMcore pose estimation
frame.

This PR changes it. We're now using the CAMERA_LINK_FRAME_* env
variables to set the base_footprint frame relative to the SLAMcore pose
estimation frame.

As part of this PR we also hardcode the transformation of the Realsense
URDF model relative to the robot base. Before we were also setting it
based on the CAMERA_LINK_FRAME_* env variables. Continuing this though
would make it impractical and we also don't gain much from an
integrator's perspective since they would have to change the URDF model
(kobuki + mounting plates + d435) altogether.

File: src/ros1_examples/descriptions/slamcore-kobuki.urdf.xacro (robot description, xacro)
@@ -6,6 +6,4 @@
        xmlns:xacro="http://ros.org/wiki/xacro">
   <xacro:arg name="camera_tf_root" default=""/>
-  <xacro:arg name="camera_link_frame_xyz" default=""/>
-  <xacro:arg name="camera_link_frame_rpy" default=""/>
   <xacro:arg name="parent_frame" default="base_footprint"/>
   <xacro:include filename="$(find kobuki_description)/urdf/kobuki.urdf.xacro" />
@@ -14,5 +12,5 @@
   <xacro:kobuki/>
   <xacro:sensor_d435 name="$(arg camera_tf_root)" parent="$(arg parent_frame)">
-    <origin xyz="$(arg camera_link_frame_xyz)" rpy="$(arg camera_link_frame_rpy)"/>
+    <origin xyz="0.09338891 0.0 0.25" rpy="0 0 0"/>
   </xacro:sensor_d435>
   <xacro:stack_mdf parent="base_link"/>

Commit message: [SCS-2659] Attach the Realsense model on the custom camera mount

File: src/ros1_examples/descriptions/slamcore-kobuki.urdf.xacro (robot description, xacro)
@@ -6,11 +6,10 @@
        xmlns:xacro="http://ros.org/wiki/xacro">
   <xacro:arg name="camera_tf_root" default=""/>
-  <xacro:arg name="parent_frame" default="base_footprint"/>
   <xacro:include filename="$(find kobuki_description)/urdf/kobuki.urdf.xacro" />
   <xacro:include filename="$(find ros1_examples)/descriptions/_d435.urdf.xacro" />
   <xacro:include filename="$(find ros1_examples)/descriptions/plates.urdf.xacro" />
   <xacro:kobuki/>
-  <xacro:sensor_d435 name="$(arg camera_tf_root)" parent="$(arg parent_frame)">
-    <origin xyz="0.09338891 0.0 0.25" rpy="0 0 0"/>
+  <xacro:sensor_d435 name="$(arg camera_tf_root)" parent="camera_mount_link">
+    <origin xyz="0.000 0.000 0.014" rpy="0.000 0.000 0.000"/>
   </xacro:sensor_d435>
   <xacro:stack_mdf parent="base_link"/>
