Commit message: [PROD-115] update package name and refs

File: src/slamcore_ros1_examples/descriptions/_d435.urdf.xacro (robot description, xacro)
@@ -45,5 +45,5 @@
       <origin xyz="${d435_cam_mount_from_center_offset} ${-d435_cam_depth_py} 0" rpy="${M_PI/2} 0 ${M_PI/2}"/>
         <geometry>
-	        <mesh filename="package://ros1_examples/meshes/d435.dae" />
+	        <mesh filename="package://slamcore_ros1_examples/meshes/d435.dae" />
         </geometry>
         <material name="${name}_aluminum"/>

File: src/slamcore_ros1_examples/descriptions/plates.urdf.xacro (robot description, xacro)
@@ -28,5 +28,5 @@
         <origin xyz="0 0 0" rpy="0 0 0"/>
         <geometry>
-          <mesh filename="package://ros1_examples/meshes/L10_standoff.stl" scale="${M_SCALE} ${M_SCALE} ${M_SCALE}"/> <!-- Small standoff STL -->
+          <mesh filename="package://slamcore_ros1_examples/meshes/L10_standoff.stl" scale="${M_SCALE} ${M_SCALE} ${M_SCALE}"/> <!-- Small standoff STL -->
         </geometry>
         <material name="ss"/>
@@ -50,5 +50,5 @@
         <origin xyz="0 0 0" rpy="0 0 0"/>
         <geometry>
-          <mesh filename="package://ros1_examples/meshes/L50_standoff.stl" scale="${M_SCALE} ${M_SCALE} ${M_SCALE}"/> <!-- Middle standoff STL -->
+          <mesh filename="package://slamcore_ros1_examples/meshes/L50_standoff.stl" scale="${M_SCALE} ${M_SCALE} ${M_SCALE}"/> <!-- Middle standoff STL -->
         </geometry>
         <material name="ss"/>
@@ -72,5 +72,5 @@
         <origin xyz=" 0 0 0" rpy="0 0 0"/>
         <geometry>
-          <mesh filename="package://ros1_examples/meshes/L50_standoff.stl" scale="${M_SCALE} ${M_SCALE} ${M_SCALE}"/> <!-- Top standoff STL -->
+          <mesh filename="package://slamcore_ros1_examples/meshes/L50_standoff.stl" scale="${M_SCALE} ${M_SCALE} ${M_SCALE}"/> <!-- Top standoff STL -->
         </geometry>
         <material name="ss"/>
@@ -107,5 +107,5 @@
         <origin xyz="0 0 0" rpy="0 0 0"/>
         <geometry>
-          <mesh filename="package://ros1_examples/meshes/bottom_plate.stl" scale="${M_SCALE} ${M_SCALE} ${M_SCALE}"/> <!-- Bottom Plate STL -->
+          <mesh filename="package://slamcore_ros1_examples/meshes/bottom_plate.stl" scale="${M_SCALE} ${M_SCALE} ${M_SCALE}"/> <!-- Bottom Plate STL -->
         </geometry>
         <material name="mdf"/>
@@ -114,5 +114,5 @@
         <origin xyz="0 0 0" rpy="0 0 0"/>
         <geometry>
-          <mesh filename="package://ros1_examples/meshes/bottom_plate.stl"
+          <mesh filename="package://slamcore_ros1_examples/meshes/bottom_plate.stl"
                 scale="${M_SCALE} ${M_SCALE} ${M_SCALE}"/>
         </geometry>
@@ -134,5 +134,5 @@
         <origin xyz="0 0 0" rpy="0 0 0"/>
         <geometry>
-          <mesh filename="package://ros1_examples/meshes/middle_plate.stl" scale="${M_SCALE} ${M_SCALE} ${M_SCALE}"/> <!-- Middle Plate STL -->
+          <mesh filename="package://slamcore_ros1_examples/meshes/middle_plate.stl" scale="${M_SCALE} ${M_SCALE} ${M_SCALE}"/> <!-- Middle Plate STL -->
         </geometry>
         <material name="mdf"/>
@@ -141,5 +141,5 @@
         <origin xyz="0.0 0.0 0.0" rpy="0 0 0"/>
         <geometry>
-          <mesh filename="package://ros1_examples/meshes/middle_plate.stl"
+          <mesh filename="package://slamcore_ros1_examples/meshes/middle_plate.stl"
                 scale="${M_SCALE} ${M_SCALE} ${M_SCALE}"/>
         </geometry>
@@ -159,5 +159,5 @@
         <origin xyz="0 0 0" rpy="0 0 0"/>
         <geometry>
-          <mesh filename="package://ros1_examples/meshes/top_plate.stl" scale="${M_SCALE} ${M_SCALE} ${M_SCALE}"/> <!-- Top Plate STL -->
+          <mesh filename="package://slamcore_ros1_examples/meshes/top_plate.stl" scale="${M_SCALE} ${M_SCALE} ${M_SCALE}"/> <!-- Top Plate STL -->
         </geometry>
         <material name="mdf"/>
@@ -166,5 +166,5 @@
         <origin xyz="0 0 0" rpy="0 0 0"/>
         <geometry>
-          <mesh filename="package://ros1_examples/meshes/top_plate.stl" scale="${M_SCALE} ${M_SCALE} ${M_SCALE}"/>
+          <mesh filename="package://slamcore_ros1_examples/meshes/top_plate.stl" scale="${M_SCALE} ${M_SCALE} ${M_SCALE}"/>
         </geometry>
       </collision>
@@ -179,5 +179,5 @@
         <origin xyz="0 0 0" rpy="0 0 0"/>
         <geometry>
-          <mesh filename="package://ros1_examples/meshes/d435i_mount.stl" scale="${M_SCALE} ${M_SCALE} ${M_SCALE}"/> <!-- Camera mount STL -->
+          <mesh filename="package://slamcore_ros1_examples/meshes/d435i_mount.stl" scale="${M_SCALE} ${M_SCALE} ${M_SCALE}"/> <!-- Camera mount STL -->
         </geometry>
         <material name="pla"/>
@@ -186,5 +186,5 @@
         <origin xyz="0 0 0" rpy="0 0 0"/>
         <geometry>
-          <mesh filename="package://ros1_examples/meshes/d435i_mount.stl" scale="${M_SCALE} ${M_SCALE} ${M_SCALE}"/>
+          <mesh filename="package://slamcore_ros1_examples/meshes/d435i_mount.stl" scale="${M_SCALE} ${M_SCALE} ${M_SCALE}"/>
         </geometry>
       </collision>

File: src/slamcore_ros1_examples/descriptions/slamcore-kobuki.urdf.xacro (robot description, xacro)
@@ -7,6 +7,6 @@
   <xacro:arg name="camera_tf_root" default=""/>
   <xacro:include filename="$(find kobuki_description)/urdf/kobuki.urdf.xacro" />
-  <xacro:include filename="$(find ros1_examples)/descriptions/_d435.urdf.xacro" />
-  <xacro:include filename="$(find ros1_examples)/descriptions/plates.urdf.xacro" />
+  <xacro:include filename="$(find slamcore_ros1_examples)/descriptions/_d435.urdf.xacro" />
+  <xacro:include filename="$(find slamcore_ros1_examples)/descriptions/plates.urdf.xacro" />
   <xacro:kobuki/>
   <xacro:sensor_d435 name="$(arg camera_tf_root)" parent="camera_mount_link">
